Commit message: Complete implementation of Physical AI textbook with capstone project

File: book/examples/humanoid-sim/gazebo_models/humanoid_simple.urdf (robot description, URDF)
Before this commit: robot humanoid_simple, 18 links, 17 joints
Links:
- removed link camera_link
- removed link left_arm_lower
- removed link left_arm_upper
- removed link left_calf
- removed link left_foot
- removed link left_hand
- removed link left_thigh
- removed link left_wrist
- removed link right_arm_lower
- removed link right_arm_upper
- removed link right_calf
- removed link right_foot
- removed link right_hand
- removed link right_thigh
- removed link right_wrist
- removed link world
- added link left_upper_arm, mass 1.5; collision cylinder length=0.4 radius=0.05; visual cylinder length=0.4 radius=0.05
- added link left_upper_leg, mass 3; collision cylinder length=0.5 radius=0.07; visual cylinder length=0.5 radius=0.07
- added link right_upper_arm, mass 1.5; collision cylinder length=0.4 radius=0.05; visual cylinder length=0.4 radius=0.05
- added link right_upper_leg, mass 3; collision cylinder length=0.5 radius=0.07; visual cylinder length=0.5 radius=0.07
- link head: mass 2.0 -> 2; geometry collision sphere radius=0.15; visual sphere radius=0.15
- link torso: mass 15.0 -> 10; geometry collision box size=0.4 0.6 0.2; visual box size=0.4 0.6 0.2
Joints:
- removed joint camera_joint
- removed joint left_ankle_pitch
- removed joint left_elbow_pitch
- removed joint left_gripper
- removed joint left_hip_pitch
- removed joint left_knee_pitch
- removed joint left_shoulder_pitch
- removed joint left_wrist_pitch
- removed joint neck_yaw
- removed joint right_ankle_pitch
- removed joint right_elbow_pitch
- removed joint right_gripper
- removed joint right_hip_pitch
- removed joint right_knee_pitch
- removed joint right_shoulder_pitch
- removed joint right_wrist_pitch
- removed joint world_to_torso
- added joint left_hip: type revolute, parent torso, child left_upper_leg, origin xyz=0 0.15 -0.1 rpy=1.5707 0 0, axis 0 0 1, limit lower=-1.57 upper=1.57 effort=20 velocity=1
- added joint left_shoulder: type revolute, parent torso, child left_upper_arm, origin xyz=0 0.35 0 rpy=1.5707 0 0, axis 0 0 1, limit lower=-1.57 upper=1.57 effort=10 velocity=1
- added joint neck: type revolute, parent torso, child head, origin xyz=0 0 0.15 rpy=0 0 0, axis 0 0 1, limit lower=-1.57 upper=1.57 effort=10 velocity=1
- added joint right_hip: type revolute, parent torso, child right_upper_leg, origin xyz=0 -0.15 -0.1 rpy=1.5707 0 0, axis 0 0 1, limit lower=-1.57 upper=1.57 effort=20 velocity=1
- added joint right_shoulder: type revolute, parent torso, child right_upper_arm, origin xyz=0 -0.35 0 rpy=-1.5707 0 0, axis 0 0 1, limit lower=-1.57 upper=1.57 effort=10 velocity=1
